Commit message: updatedd pybullet model

File: ur5_pybullet.urdf (robot description, URDF)
Before this commit: robot ur5, 7 links, 6 joints
Links:
- link base_link: geometry collision cylinder length=0.1 radius=0.08; visual mesh filename=meshes/visual/base.stl scale=1 1 1
- link forearm_link: geometry collision cylinder length=0.39225 radius=0.045; visual mesh filename=meshes/visual/forearm.stl scale=1 1 1
- link shoulder_link: geometry collision cylinder length=0.1 radius=0.06; visual mesh filename=meshes/visual/shoulder.stl scale=1 1 1
- link upper_arm_link: geometry collision cylinder length=0.425 radius=0.05; visual mesh filename=meshes/visual/upperarm.stl scale=1 1 1
- link wrist_1_link: geometry collision cylinder length=0.08 radius=0.035; visual mesh filename=meshes/visual/wrist1.stl scale=1 1 1
- link wrist_2_link: geometry collision cylinder length=0.08 radius=0.035; visual mesh filename=meshes/visual/wrist2.stl scale=1 1 1
- link wrist_3_link: geometry collision cylinder length=0.06 radius=0.03; visual mesh filename=meshes/visual/wrist3.stl scale=1 1 1
